Commit message: commented out unused links in UM_MRZR.urdf

File: avt_341/config/UM_MRZR.urdf (robot description, URDF)
Before this commit: robot MRZR, 9 links, 8 joints
Links:
- removed link flir_optical
- removed link os_lidar
- removed link os_sensor
- removed link vbox_link
- removed link vectornav_link
- removed link vlp16_top_link
Joints:
- removed joint os_sensor_to_flir_optical
- removed joint vbox_to_front_diff
- removed joint vectornav_to_front_diff
- removed joint vlp16_top_to_front_diff
- removed joint vlp16_top_to_os_lidar
- removed joint vlp16_top_to_os_sensor
