Commit message: Added yaw rate limiter to speed_control_node

File: avt_341/config/MRZR_UE.urdf (robot description, URDF)
Before this commit: robot MRZR, 8 links, 7 joints
Joints:
- joint vlp16_top_to_os_sensor: origin xyz=0.0 0.0 0.0 rpy=0.0 -0.017453292519943295 -0.06981317007977318 -> xyz=0.0 0.0 0.0 rpy=0.0 0.0 0.0

Commit message: Added lidar obstacle detection for ROS2

File: avt_341/config/MRZR_UE.urdf (robot description, URDF)
Before this commit: robot MRZR, 9 links, 8 joints
Links:
- removed link flir_optical
Joints:
- removed joint os_sensor_to_flir_optical
- joint vlp16_top_to_os_sensor: origin xyz=0.0 0.0 0.0 rpy=0.0 -0.017453292519943295 -0.06981317007977318 -> xyz=0.0 0.0 0.0 rpy=0.0 0.0 0.0
