Commit message: Fixed bug with control node driving when no valid plans are available.

File: avt_341/config/MRZR.urdf (robot description, URDF)
Before this commit: robot MRZR, 9 links, 8 joints
Links:
- link front_diff_link: geometry 

Commit message: Added intermediate point generation to global planner

File: avt_341/config/MRZR.urdf (robot description, URDF)
Before this commit: robot MRZR, 9 links, 8 joints
Links:
- removed link odom
Joints:
- removed joint odom_to_vectornav

Commit message: Build fixes, added flir_optical frame and transform to lidar to MRZR.urdf

File: avt_341/config/MRZR.urdf (robot description, URDF)
Before this commit: robot MRZR, 8 links, 7 joints
Links:
- added link flir_optical
Joints:
- added joint os_sensor_to_flir_optical: type fixed, parent os_sensor, child flir_optical, origin xyz=-0.283517 0.0682941 -0.136282 rpy=-1.481708200033002 -0.017688723295176803 1.5783145437948567

Commit message: Updated to default ROS camera calibration format

File: avt_341/config/MRZR.urdf (robot description, URDF)
Before this commit: robot MRZR, 9 links, 8 joints
Joints:
- removed joint os_sensor_to_flir_optical

Commit message: Minor fixes to calibration publisher

File: avt_341/config/MRZR.urdf (robot description, URDF)
Before this commit: robot MRZR, 9 links, 7 joints
Links:
- removed link flir_optical

Commit message: Updated static transform for FLIR camera optical frame

File: avt_341/config/MRZR.urdf (robot description, URDF)
Before this commit: robot MRZR, 9 links, 8 joints
Joints:
- removed joint vlp16_top_to_os_lidar
- joint os_sensor_to_flir_optical: parent os_sensor -> os_lidar

Commit message: Fixes to KRC MRZR tf tree

File: avt_341/config/MRZR.urdf (robot description, URDF)
Before this commit: robot MRZR, 9 links, 8 joints
Links:
- removed link flir_optical
- removed link os_lidar
Joints:
- removed joint os_sensor_to_flir_optical
- removed joint vlp16_top_to_os_lidar

Commit message: update MRZR1 urdf and static frames

File: avt_341/config/MRZR.urdf (robot description, URDF)
Before this commit: robot MRZR, 9 links, 8 joints
Links:
- removed link base_link
- removed link flir_optical
- removed link front_diff_link
- removed link os_lidar
- removed link os_sensor
- removed link rear_diff_link
- removed link vbox_link
- removed link vectornav_link
- removed link vlp16_top_link
- added link cg_link; visual box size=2.71 2.59 2
Joints:
- removed joint front_diff_to_base
- removed joint os_sensor_to_flir_optical
- removed joint rear_diff_to_front_diff
- removed joint vbox_to_front_diff
- removed joint vectornav_to_front_diff
- removed joint vlp16_top_to_front_diff
- removed joint vlp16_top_to_os_lidar
- removed joint vlp16_top_to_os_sensor

Commit message: Added vectornav transform

File: avt_341/config/MRZR.urdf (robot description, URDF)
Before this commit: robot MRZR, 9 links, 8 joints
Joints:
- joint vectornav_to_front_diff: origin xyz=-1.30526 0.00114614 1.55394 rpy=0.008775322550313533 -0.04598729640809592 -0.03823053204542514 -> xyz=-1.30526 0.00114614 1.55394 rpy=0.008775322550313533 -0.04598729640809592 -1.6090268588403216
